File: VibeDeck.kicad_sch (KiCad schematic)
At the start: 21 parts, among them J1 Conn_01x04, SW1 SW_Push, SW10 RotaryEncoder_Switch, SW2 SW_Push, SW3 SW_Push, SW4 SW_Push, SW5 SW_Push, SW6 SW_Push, SW7 SW_Push, SW8 SW_Push, SW9 SW_Push, U1 MOUDLE-SEEEDUINO-XIAO

Commit message: Add files via upload
Connections:
- net 3V3: now also U1.12 (3V3)
- net GND: now also U1.13 (GND)
- net SCL: now also U1.6 (PA9_A5_D5_SCL)
- net SDA: now also U1.5 (PA8_A4_D4_SDA)
Changed lines of the file:
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@@
+		)
+	)
+	(label "3V3"
+		(at 76.2 83.82 0)
+		(effects
+			(font
+				(size 1.27 1.27)
+			)
+			(justify left bottom)
 		)
 	)
@@
 		)
 	)
+	(label "GND"
+		(at 76.2 81.28 0)
+		(effects
+			(font
+				(size 1.27 1.27)
+			)
+			(justify left bottom)
+		)
+	)
 	(label "ROW1"
 		(at 190.5 76.2 0)
@@
 		)
 	)
+	(label "SCL"
+		(at 35.56 91.44 0)
+		(effects
+			(font
+				(size 1.27 1.27)
+			)
+			(justify left bottom)
+		)
+	)
 	(label "ENC_A"
 		(at 129.54 35.56 0)
 		(effects
 			(font
+				(size 1.27 1.27)
+			)
+			(justify left bottom)
+		)
+	)
+	(label "SDA"
+		(at 35.56 88.9 0)
+		(effects
+			(font
